Commit message: Atualiza repositório

File: bumperbot_ws/src/bumperbot_description/urdf/bumperbot.urdf.xacro (robot description, xacro)
@@ -197,9 +197,63 @@
   </inertial>
 </link>
-  <joint name="antena_joint" type="fixed">
-    <origin xyz="0 0 0.1" rpy="0 0 0" />
+  <joint name="antena_joint_1" type="fixed">
+    <origin xyz="0 -0.01 0.1" rpy="0 0 0" />
     <parent link="base_link" />
     <child link="antenna_1_link" />
     <axis xyz="0 0 0" />
   </joint>
+<link name="antenna_2_link">
+  <visual>
+    <origin xyz="0 0.00 0" rpy="0 0 0"/>
+      <geometry> <mesh filename="package://bumperbot_description/models/antenna_1/meshes/antenna_visual.stl" scale="0.3 0.1 0.3"/>
+</geometry>
+    <material name="light_black"/>
+  </visual>
+  <collision>
+    <origin xyz="0 0.00 0.000" rpy="0 0 0"/>
+    <geometry>
+      <box size="0.140 0.140 0.143"/>
+    </geometry>
+  </collision>
+  <inertial>
+    <origin xyz="0 0 0" rpy="0 0 0"/>
+    <mass value="0.2573504e-01"/>
+    <inertia ixx="2.2124416e-03" ixy="-1.2294101e-05" ixz="3.4938785e-05"
+             iyy="2.1193702e-03" iyz="-5.0120904e-06"
+             izz="2.0064271e-03" />
+  </inertial>
+</link>
+  <joint name="antena_joint_2" type="fixed">
+    <origin xyz="0 0.01 0.1" rpy="0 0 0" />
+    <parent link="base_link" />
+    <child link="antenna_2_link" />
+    <axis xyz="0 0 0" />
+  </joint>
+<link name="antenna_3_link">
+  <visual>
+    <origin xyz="0 0.00 0" rpy="0 0 0"/>
+      <geometry> <mesh filename="package://bumperbot_description/models/antenna_1/meshes/antenna_visual.stl" scale="0.3 0.1 0.3"/>
+</geometry>
+    <material name="light_black"/>
+  </visual>
+  <collision>
+    <origin xyz="0 0.00 0.000" rpy="0 0 0"/>
+    <geometry>
+      <box size="0.140 0.140 0.143"/>
+    </geometry>
+  </collision>
+  <inertial>
+    <origin xyz="0 0 0" rpy="0 0 0"/>
+    <mass value="0.2573504e-01"/>
+    <inertia ixx="2.2124416e-03" ixy="-1.2294101e-05" ixz="3.4938785e-05"
+             iyy="2.1193702e-03" iyz="-5.0120904e-06"
+             izz="2.0064271e-03" />
+  </inertial>
+</link>
+  <joint name="antena_joint_3" type="fixed">
+    <origin xyz="-0.01 0 0.1" rpy="0 0 0" />
+    <parent link="base_link" />
+    <child link="antenna_3_link" />
+    <axis xyz="0 0 0" />
+  </joint>
 </robot>

File: bumperbot_ws/src/bumperbot_description/urdf/bumperbot_gazebo.xacro (robot description, xacro)
@@ -81,6 +81,6 @@
          <parent_frame>world</parent_frame>
          <tags_per_fix>5</tags_per_fix>
-         <fix_sdf_path>/home/ropingoold/agricultural_automotion_robot/bumperbot_ws/src/bumperbot_description/models/normal_size_fixture/model.sdf</fix_sdf_path>
-         <tag_sdf_path>/home/ropingoold/agricultural_automotion_robot/bumperbot_ws/src/bumperbot_description/models/antenna_1/model.sdf</tag_sdf_path>
+         <fix_sdf_path>/home/ropingoold/Self-Driving-and-ROS-Learn-by-Doing-Odometry-Control/Section11_Sensor-Fusion/bumperbot_ws/src/bumperbot_description/models/normal_size_fixture/model.sdf</fix_sdf_path>
+         <tag_sdf_path>/home/ropingoold/Self-Driving-and-ROS-Learn-by-Doing-Odometry-Control/Section11_Sensor-Fusion/bumperbot_ws/src/bumperbot_description/models/antenna_1/model.sdf</tag_sdf_path>
        </plugin>
      </sensor>
@@ -92,13 +92,55 @@
        <tag_name>rfid_tag1</tag_name>
        <detected_tag_name>rfid_tag_1</detected_tag_name>
-       <detected_tag_colour>blue</detected_tag_colour>
+      <bodyName>antenna_1_link</bodyName>
+      <frameName>antenna_1_link</frameName>
+       <!-- <detected_tag_colour>blue</detected_tag_colour> -->
        <antenna_id>1</antenna_id>
        <azimuth_beamwidth>1</azimuth_beamwidth>
        <elevation_beamwidth>1</elevation_beamwidth>
        <rzero>2</rzero>
-       <tag_yellow_sdf_path>/home/ropingoold/agricultural_automotion_robot/bumperbot_ws/src/bumperbot_description/models/RFID_3/model.sdf</tag_yellow_sdf_path>
-      <tag_red_sdf_path>/home/ropingoold/agricultural_automotion_robot/bumperbot_ws/src/bumperbot_description/models/RFID_2/model.sdf</tag_red_sdf_path>
-      <tag_blue_sdf_path>/home/ropingoold/agricultural_automotion_robot/bumperbot_ws/src/bumperbot_description/models/RFID_5/model.sdf</tag_blue_sdf_path>
-      <tag_purple_sdf_path>/home/ropingoold/agricultural_automotion_robot/bumperbot_ws/src/bumperbot_description/models/RFID_4/model.sdf</tag_purple_sdf_path>
+       <tag_yellow_sdf_path>/home/ropingoold/Self-Driving-and-ROS-Learn-by-Doing-Odometry-Control/Section11_Sensor-Fusion/bumperbot_ws/src/bumperbot_description/models/RFID_3/model.sdf</tag_yellow_sdf_path>
+      <tag_red_sdf_path>/home/ropingoold/Self-Driving-and-ROS-Learn-by-Doing-Odometry-Control/Section11_Sensor-Fusion/bumperbot_ws/src/bumperbot_description/models/RFID_2/model.sdf</tag_red_sdf_path>
+      <tag_blue_sdf_path>/home/ropingoold/Self-Driving-and-ROS-Learn-by-Doing-Odometry-Control/Section11_Sensor-Fusion/bumperbot_ws/src/bumperbot_description/models/RFID_5/model.sdf</tag_blue_sdf_path>
+      <tag_purple_sdf_path>/home/ropingoold/Self-Driving-and-ROS-Learn-by-Doing-Odometry-Control/Section11_Sensor-Fusion/bumperbot_ws/src/bumperbot_description/models/RFID_4/model.sdf</tag_purple_sdf_path>
+     </plugin>
+   </sensor>
+</gazebo>
+<gazebo reference="base_link">
+      <sensor type="rfid" name="rfid_antenna_2">
+     <plugin name="rfid_antenna_2" filename="libRFID_antenna_plugin.so">
+       <antenna_name>antenna_2</antenna_name>
+        <bodyName>antenna_2_link</bodyName>
+      <frameName>antenna_2_link</frameName>
+       <tag_name>rfid_tag2</tag_name>
+       <detected_tag_name>rfid_tag_2</detected_tag_name>
+       <!-- <detected_tag_colour>red</detected_tag_colour> -->
+       <antenna_id>2</antenna_id>
+       <azimuth_beamwidth>1</azimuth_beamwidth>
+       <elevation_beamwidth>1</elevation_beamwidth>
+       <rzero>2</rzero>
+       <tag_yellow_sdf_path>/home/ropingoold/Self-Driving-and-ROS-Learn-by-Doing-Odometry-Control/Section11_Sensor-Fusion/bumperbot_ws/src/bumperbot_description/models/RFID_3/model.sdf</tag_yellow_sdf_path>
+      <tag_red_sdf_path>/home/ropingoold/Self-Driving-and-ROS-Learn-by-Doing-Odometry-Control/Section11_Sensor-Fusion/bumperbot_ws/src/bumperbot_description/models/RFID_2/model.sdf</tag_red_sdf_path>
+      <tag_blue_sdf_path>/home/ropingoold/Self-Driving-and-ROS-Learn-by-Doing-Odometry-Control/Section11_Sensor-Fusion/bumperbot_ws/src/bumperbot_description/models/RFID_5/model.sdf</tag_blue_sdf_path>
+      <tag_purple_sdf_path>/home/ropingoold/Self-Driving-and-ROS-Learn-by-Doing-Odometry-Control/Section11_Sensor-Fusion/bumperbot_ws/src/bumperbot_description/models/RFID_4/model.sdf</tag_purple_sdf_path>
+     </plugin>
+   </sensor>
+</gazebo>
+   <gazebo reference="base_link">
+      <sensor type="rfid" name="rfid_antenna_3">
+     <plugin name="rfid_antenna_3" filename="libRFID_antenna_plugin.so">
+       <antenna_name>antenna_3</antenna_name>
+       <tag_name>rfid_tag3</tag_name>
+        <bodyName>antenna_3_link</bodyName>
+      <frameName>antenna_3_link</frameName>
+       <detected_tag_name>rfid_tag_3</detected_tag_name>
+       <!-- <detected_tag_colour>yellow</detected_tag_colour> -->
+       <antenna_id>3</antenna_id>
+       <azimuth_beamwidth>1</azimuth_beamwidth>
+       <elevation_beamwidth>1</elevation_beamwidth>
+       <rzero>2</rzero>
+       <tag_yellow_sdf_path>/home/ropingoold/Self-Driving-and-ROS-Learn-by-Doing-Odometry-Control/Section11_Sensor-Fusion/bumperbot_ws/src/bumperbot_description/models/RFID_3/model.sdf</tag_yellow_sdf_path>
+      <tag_red_sdf_path>/home/ropingoold/Self-Driving-and-ROS-Learn-by-Doing-Odometry-Control/Section11_Sensor-Fusion/bumperbot_ws/src/bumperbot_description/models/RFID_2/model.sdf</tag_red_sdf_path>
+      <tag_blue_sdf_path>/home/ropingoold/Self-Driving-and-ROS-Learn-by-Doing-Odometry-Control/Section11_Sensor-Fusion/bumperbot_ws/src/bumperbot_description/models/RFID_5/model.sdf</tag_blue_sdf_path>
+      <tag_purple_sdf_path>/home/ropingoold/Self-Driving-and-ROS-Learn-by-Doing-Odometry-Control/Section11_Sensor-Fusion/bumperbot_ws/src/bumperbot_description/models/RFID_4/model.sdf</tag_purple_sdf_path>
      </plugin>
    </sensor>
